File: Hardware/WaterGame.kicad_pcb (KiCad board)
At the start: 2 copper layers, 15 parts, among them J1A1 Conn_01x07, J1B1 Conn_01x07, J1C1 Conn_01x07, J2 Conn_02x04_Counter_Clockwise, J3 Conn_01x02, J4 Conn_01x02, J5A1 Conn_01x06, J5A2 Conn_01x06, U1 LM7805_TO220, U2 LD33V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

Commit message: Hardware: Final PCB
Parts:
- added G***: LOGO, graphics:logo_inverted_small, F.Cu at (86.4, 50.8)
- J2: value Conn_02x04_Counter_Clockwise -> Conn_02x04_Odd_Even
- U4: footprint Connector_PinSocket_2.54mm:PinSocket_2x04_P2.54mm_Vertical -> ESP8266:ESP-01
- moved U4 3.18 mm to (139.7, 71.5)
- moved J3 2.54 mm to (111.8, 85.1), turned to 0 degrees
- moved J4 2.54 mm to (130.8, 78.7), turned to -90 degrees
- moved J2 1.28 mm to (83.8, 81.3)
Connections:
- J2 pad 2: Net-(J2-Pad2) -> Net-(U6-Pad6)
- J2 pad 3: Net-(J2-Pad3) -> Net-(U6-Pad11)
- J2 pad 4: Net-(J2-Pad4) -> Net-(U6-Pad14)
- U2 pad 1: Net-(J3-Pad1) -> Net-(J1C1-Pad7)
- U2 pad 2: Net-(J1C1-Pad7) -> Net-(J5A2-Pad4)
- U2 pad 3: Net-(J5A2-Pad4) -> Net-(J3-Pad1)
- U5 pad 11: Net-(J2-Pad4) -> Net-(J2-Pad7)
- U5 pad 14: Net-(J2-Pad5) -> Net-(J2-Pad8)
- U5 pad 3: Net-(J2-Pad3) -> Net-(J2-Pad5)
- U6 pad 11: Net-(J2-Pad2) -> Net-(U6-Pad11)
- U6 pad 14: Net-(J2-Pad7) -> Net-(U6-Pad14)
- U6 pad 6: Net-(J2-Pad8) -> Net-(U6-Pad6)
Routing:
- net Net-(J1C1-Pad7): track 0.00 -> 159.3 mm
- net Net-(J1B1-Pad1): track 0.00 -> 110.0 mm
- net Net-(J3-Pad1): track 0.00 -> 75.9 mm, vias 0 -> 1
- net Net-(J5A2-Pad4): track 0.00 -> 62.7 mm
- net Net-(J2-Pad5): track 0.00 -> 60.0 mm
- net Net-(U3-Pad28): track 0.00 -> 52.5 mm
- net Net-(J5A1-Pad6): track 0.00 -> 44.1 mm, vias 0 -> 2
- net Net-(J5A1-Pad5): track 0.00 -> 41.7 mm, vias 0 -> 1
- net Net-(J5A2-Pad5): track 0.00 -> 38.9 mm
- net Net-(J2-Pad8): track 0.00 -> 38.2 mm
- net Net-(U3-Pad12): track 0.00 -> 35.8 mm
- net Net-(U5-Pad6): track 0.00 -> 34.8 mm
- net Net-(U3-Pad3): track 0.00 -> 30.3 mm
- net Net-(J2-Pad7): track 0.00 -> 28.6 mm
- net Net-(U3-Pad19): track 0.00 -> 28.1 mm
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Other:
- board outline added: 76.2 x 47 mm
- board text added: "- +"
- board text added: "3V3 Reg"
- board text added: "5V Reg"
- board text added: "9V G"
- board text added: "ESP8266"
- board text added: "GPIO"
- board text added: "J1"
- board text added: "J3"
- board text added: "J5"
- board text added: "Level shifter"
- board text added: "Motors"
- board text added: "POWER"
- board text added: "PWM"
- board text added: "S 5V G"
- board text added: "Water Game"
- board text added: "WiFi PRG"

Commit message: Hardware: Widened high-current traces
Connections:
- U3 pad 2: unconnected-(U3-Pad2) -> Net-(U3-Pad2)
- U5 pad 1: Net-(J1C1-Pad7) -> Net-(U3-Pad2)
Routing:
- net Net-(J1C1-Pad7): track 159.3 -> 149.9 mm
- net Net-(J3-Pad1): track 75.9 -> 83.3 mm, vias 1 -> 0
- net Net-(U3-Pad2): track 0.00 -> 6.92 mm
- net Net-(J5A2-Pad6): track 22.9 -> 26.5 mm
- net Net-(J5A1-Pad6): track 44.1 -> 47.5 mm, vias 2 -> 1
- net Net-(J5A2-Pad4): track 62.7 -> 65.6 mm
- net Net-(J1B1-Pad1): track 110.0 -> 107.5 mm
- net Net-(U6-Pad3): track 19.3 -> 17.9 mm
- net Net-(U6-Pad14): track 16.8 -> 15.8 mm
Other:
- board text added: "v1"
